File: RNS/Project/main.sch (EAGLE design)
At the start: 10 parts

Commit message: Change design to fit IMU and Power Base inside the board
Parts:
- removed MPU: (no value), MIA-Training:PINHD-1X4
- added IMU: IMU_ROBOCON_GY521, MIA_LIBRARY-2-2-2:IMU_ROBOCON_GY521
- IN_PW: device MIA-Training:PINHD-1X2 -> MIA_LIBRARY-2-2-2:PINHD-2_DATA
- renumbered J1 to JACK
Connections:
- net 3.3V: now also IMU.VCC; no longer MPU.1
- net GND: now also IMU.GND; no longer MPU.2
- net PB_12: now also ENC.4
- net PB_13: now also ENC.3
- net PB_4: no longer ENC.4
- net PB_5: no longer ENC.3
- net PB_6: now also IMU.SCL; no longer MPU.4
- net PB_7: now also IMU.SDA; no longer MPU.3
